File: Console.kicad_pcb (KiCad board)
At the start: 2 copper layers, 206 x 80 mm, 37 parts, among them J1 SWD CONN, J2 Conn_01x08_Female, J3 Micro_SD_Card, J4 USB_B_Micro, J5 Conn_01x08_Female, U1 LM1117MPX-3_3_NOPB, U2 STM32F103TBUx

Commit message: fixed problems, switched MCU with another of the same product line
Parts:
- added C9: 100nF, Capacitor_SMD:C_0402_1005Metric, F.Cu at (155.9, 103.2)
- J1: value SWD CONN -> Conn_01x06_Male; footprint Connector_PinHeader_1.27mm:PinHeader_2x05_P1.27mm_Vertical_SMD -> Connector_PinHeader_2.54mm:PinHeader_1x06_P2.54mm_Vertical
- U2: value STM32F103TBUx -> STM32F103C8Tx; footprint Package_DFN_QFN:QFN-36-1EP_6x6mm_P0.5mm_EP4.1x4.1mm -> Package_QFP:LQFP-48_7x7mm_P0.5mm
- moved C6 11.1 mm to (147.5, 94.2), turned to 0 degrees
- moved C7 8.82 mm to (152.6, 105.8), turned to 180 degrees
- moved J1 8.32 mm to (124.3, 137.8), turned to -90 degrees
- moved C8 5.97 mm to (144.2, 102.9), turned to 90 degrees
- moved R1 1.61 mm to (150.8, 108.2), turned to -90 degrees
- moved C4 1.35 mm to (151.6, 112.3)
Connections:
- J1 pad 2: SWDIO -> SWCLK
- J1 pad 4: SWCLK -> SWDIO
- J1 pad 5: GND -> NRST
- J2 pad 1: +3.3V -> GND
- J2 pad 2: GND -> +3.3V
- U2 pad 10: GPIO_CS -> GPIO_A
- U2 pad 11: SPI_CS -> GPIO_B
- U2 pad 12: SPI_SCK -> SCR_DC
- U2 pad 13: SPI_MISO -> GPIO_CS
- U2 pad 14: SPI_MOSI -> SPI_CS
- U2 pad 15: GPIO_X -> SPI_SCK
- U2 pad 16: GPIO_Y -> SPI_MISO
- U2 pad 17: unconnected-(U2-Pad17) -> SPI_MOSI
- U2 pad 18: GND -> GPIO_X
- U2 pad 19: +3.3V -> GPIO_Y
- U2 pad 20: GPIO_UP -> unconnected-(U2-Pad20)
- U2 pad 21: GPIO_LEFT -> unconnected-(U2-Pad21)
- U2 pad 22: GPIO_DOWN -> unconnected-(U2-Pad22)
- U2 pad 23: GPIO_RIGHT -> GND
- U2 pad 24: unconnected-(U2-Pad24) -> +3.3V
- U2 pad 25: SWDIO -> unconnected-(U2-Pad25)
- U2 pad 26: GND -> unconnected-(U2-Pad26)
- U2 pad 27: +3.3V -> unconnected-(U2-Pad27)
- U2 pad 28: SWCLK -> unconnected-(U2-Pad28)
- U2 pad 29: unconnected-(U2-Pad29) -> GPIO_UP
- U2 pad 30: SWO -> GPIO_LEFT
- U2 pad 31: SCR_BLK -> GPIO_DOWN
- U2 pad 32: SCR_RST -> GPIO_RIGHT
- U2 pad 34: unconnected-(U2-Pad34) -> SWDIO
- U2 pad 35: BOOT0 -> GND
- U2 pad 36: GND -> +3.3V
- U2 pad 37: unconnected-(U2-Pad37) -> SWCLK
- U2 pad 4: NRST -> unconnected-(U2-Pad4)
- U2 pad 7: GPIO_A -> NRST
- U2 pad 8: GPIO_B -> unconnected-(U2-Pad8)
- U2 pad 9: SCR_DC -> unconnected-(U2-Pad9)
Routing:
- net GND: track 420.7 -> 448.8 mm, vias 7 -> 9
- net NRST: track 49.0 -> 69.7 mm
- net +3.3V: track 417.2 -> 434.0 mm, vias 10 -> 13
- net SWO: track 39.3 -> 51.8 mm, vias 0 -> 2
- net SWDIO: track 41.0 -> 50.0 mm, vias 0 -> 2
- net SWCLK: track 39.4 -> 44.7 mm, vias 0 -> 2
- net SCR_BLK: track 42.1 -> 46.4 mm, vias 0 -> 2
- net GPIO_DOWN: track 96.7 -> 94.1 mm
- net SCR_RST: track 41.4 -> 43.9 mm, vias 0 -> 4
- net GPIO_RIGHT: track 68.3 -> 66.0 mm
- net GPIO_LEFT: track 120.6 -> 118.5 mm, vias 2 -> 0
- net GPIO_B: track 91.5 -> 89.5 mm
- net SPI_MISO: track 38.2 -> 36.5 mm
- net BOOT0: track 4.80 -> 3.17 mm, vias 2 -> 0
- net SPI_SCK: track 75.7 -> 74.1 mm
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